File: Scheme/schemat.sch (EAGLE design)
At the start: 15 parts, among them IC1 7805T

Commit message: schemat v2
Parts:
- added M1: ARDUINO-NANO-3.0, diy-modules:ARDUINO-NANO-3.0
- added U$10: SUNLOGO, adafruit:SUNLOGO
- U$1: value NANO -> (none); device Arduino-clone:NANO -> keypad4x4_ece:KEYPAD4X4
Connections:
- removed net 12V: R1.1, U$1.RAW, U$2.TIP
- removed net 5V: C2.1, IC1.VO, U$3.VCC
- removed net N$1 (its old number): U$4.VCC
- removed net N$21: U$5.VCC
- removed net N$22: U$3.SCL
- removed net N$23: U$5.OUT
- removed net N$24: U$6.VCC
- removed net N$25: U$6.OUT
- removed net N$26: U$7.VCC
- removed net N$27: U$7.OUT
- removed net N$28: U$8.VCC
- removed net N$29: U$8.OUT
- removed net N$3: C1.+, IC1.VI, LED1.C
- removed net N$32: U$9.IN2
- removed net N$33: U$9.VCC.1
- removed net N$4: U$4.OUT
- new net +5V: C2.1, IC1.VO, U$3.VCC, U$4.VCC, U$5.VCC, U$6.VCC, U$7.VCC, U$8.VCC, U$9.VCC.1
- new net KEY1: M1.D4, U$1.R1
- new net KEY2: M1.D5, U$1.R2
- new net KEY3: M1.D6, U$1.R3
- new net KEY4: M1.D7, U$1.R4
- new net KEY5: M1.D8, U$1.C1
- new net KEY6: M1.D9, U$1.C2
- new net KEY7: M1.D10, U$1.C3
- new net KEY8: M1.D11/MOSI, U$1.C4
- new net PIR1: M1.A2, U$4.OUT
- new net PIR2: M1.D0/RX, U$5.OUT
- new net PIR3: M1.D1/TX, U$6.OUT
- new net PIR4: M1.D2, U$7.OUT
- new net PIR5: M1.D3, U$8.OUT
- new net SDA: M1.A4, U$3.SDA
- new net VCC: C1.+, IC1.VI, M1.VIN, R1.1, U$2.TIP
- net GND: now also LED1.C, M1.GND.1, M1.GND.2; no longer U$1.GND
- net RELAY1: now also M1.A0
- net SCL: now also M1.A5, U$3.SCL; no longer U$3.SDA
Other:
- moved on the sheet: C1, C2, IC1, LED1, R1, U$4, U$5, U$6, U$7, U$8, U$9
